File: board/MINI_SAM_TQFP_2.54_BB_2017_01_17_004.brd (EAGLE design)
At the start: 24.1 x 39.2 mm, 29 parts, among them J1 MOLEX_47346-100147346, J2 CORTEX_DEBUGPTH, SW1 KMS_SWITCHKMS, SW2 KMS_SWITCHKMS, U1 SAMD21ETQFP, Y1 32.768kHz 7pF

Commit message: Add files via upload
Parts:
- LED: device microbuilder:CHIPLED_0603_NOOUTLINE -> microbuilder:CHIPLED_0805_NOOUTLINE
- moved L/EN 0.96 mm to (6.15, 25.9), turned to 90 degrees
- moved LED 0.15 mm to (7.70, 25.0), turned to 180 degrees
Routing:
- net LED: track 4.27 -> 6.39 mm
- net N$2: track 2.98 -> 1.76 mm
- net SWCLK: track 13.5 -> 14.6 mm
Changed lines of the file:
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@@
 <attribute name="VALUE" x="4.96" y="0.13" size="0.4064" layer="28" ratio="10" rot="MR90"/>
 </element>
-<element name="LED" library="microbuilder" package="CHIPLED_0603_NOOUTLINE" value="APT2012LSECK/J3-PRV" x="7.55" y="25" smashed="yes">
-<attribute name="NAME" x="7.55" y="26.42" size="0.6096" layer="25" font="vector" ratio="18" align="bottom-center"/>
+<element name="LED" library="microbuilder" package="CHIPLED_0805_NOOUTLINE" value="APT2012LSECK/J3-PRV" x="7.7" y="25" smashed="yes" rot="R180">
+<attribute name="NAME" x="7.7" y="26.77" size="0.6096" layer="25" font="vector" ratio="18" align="bottom-center"/>
 </element>
 <element name="IC1" library="Shockley_Custom" package="SOT23" value="" x="19.9" y="23.2" smashed="yes" rot="R27.7">
@@
 <element name="SW1" library="Shockley_Custom" package="KMS_SWITCH" value="KMS_SWITCHKMS" x="8.075" y="1.8" smashed="yes"/>
 <element name="R1" library="Shockley_Custom" package="CAT16_ARRAY" value="RESISTOR_ARRAY_4CAT16" x="10.4" y="25" rot="R180"/>
-<element name="L/EN" library="SparkFun-Jumpers" package="SMT-JUMPER_2_NO_NO-SILK" value="JUMPER-SMT_2_NO_NO-SILK" x="6" y="25" smashed="yes">
-<attribute name="NAME" x="6" y="25.843" size="0.5" layer="25" font="vector" ratio="18" align="bottom-center"/>
+<element name="L/EN" library="SparkFun-Jumpers" package="SMT-JUMPER_2_NO_NO-SILK" value="JUMPER-SMT_2_NO_NO-SILK" x="6.15" y="25.95" smashed="yes" rot="R90">
+<attribute name="NAME" x="5.307" y="25.95" size="0.5" layer="25" font="vector" ratio="18" rot="R90" align="bottom-center"/>
 </element>
 <element name="JP5" library="Shockley_Custom" package="SMD2.5MMX1.5MM" value="FR11_PAD2.5MMX1.5MM" x="17.7" y="1.3" rot="MR90"/>
@@
 <contactref element="SW2" pad="3"/>
 <contactref element="SW2" pad="4"/>
+<via x="7.7" y="22.95" extent="1-16" drill="0.3"/>
 </signal>
 <signal name="USBD+" class="1">
@@
 <contactref element="R1" pad="5"/>
 <wire x1="9.2" y1="24.15" x2="9.2" y2="23.9" width="0.254" layer="1"/>
-<wire x1="4.197384375" y1="21.374859375" x2="6.424859375" y2="21.374859375" width="0.254" layer="1"/>
-<wire x1="6.424859375" y1="21.374859375" x2="9.2" y2="24.15" width="0.254" layer="1"/>
 <wire x1="7.4" y1="15.9" x2="7.4" y2="18.17224375" width="0.254" layer="2"/>
 <wire x1="7.4" y1="18.17224375" x2="4.197384375" y2="21.374859375" width="0.254" layer="2"/>
+<wire x1="6.95" y1="24.85" x2="8.5" y2="24.85" width="0.254" layer="1"/>
+<wire x1="8.5" y1="24.85" x2="9.2" y2="24.15" width="0.254" layer="1"/>
+<wire x1="6.95" y1="24.85" x2="5.75" y2="23.65" width="0.254" layer="1"/>
+<wire x1="5.75" y1="23.65" x2="5.75" y2="22.75" width="0.254" layer="1"/>
+<wire x1="5.75" y1="22.75" x2="4.374859375" y2="21.374859375" width="0.254" layer="1"/>
+<wire x1="4.374859375" y1="21.374859375" x2="4.197384375" y2="21.374859375" width="0.254" layer="1"/>
 </signal>
 <signal name="SWDIO">
@@
 <wire x1="7.7074" y1="15.1" x2="8.3" y2="15.1" width="0.2032" layer="1"/>
 <contactref element="J2" pad="2"/>
-<wire x1="8.3" y1="15.1" x2="8.3" y2="19.6" width="0.254" layer="2"/>
-<wire x1="8.3" y1="19.6" x2="5.266296875" y2="22.633703125" width="0.254" layer="2"/>
-<wire x1="5.266296875" y1="22.633703125" x2="4.36535" y2="22.633703125" width="0.254" layer="2"/>
+<wire x1="8.3" y1="15.1" x2="8.3" y2="19.25" width="0.254" layer="2"/>
+<wire x1="8.3" y1="19.25" x2="4.916296875" y2="22.633703125" width="0.254" layer="2"/>
+<wire x1="4.916296875" y1="22.633703125" x2="4.36535" y2="22.633703125" width="0.254" layer="2"/>
 </signal>
 <signal name="28">
@@
 <contactref element="R1" pad="3"/>
 <contactref element="L/EN" pad="2"/>
-<wire x1="6.4064" y1="25" x2="9.7" y2="25" width="0.254" layer="1"/>
-<wire x1="9.7" y1="25" x2="10" y2="25.3" width="0.254" layer="1"/>
 <wire x1="10" y1="25.3" x2="10" y2="25.85" width="0.254" layer="1"/>
+<wire x1="8.4" y1="27" x2="8.65" y2="26.75" width="0.254" layer="1"/>
+<wire x1="8.65" y1="26.75" x2="8.65" y2="25.3" width="0.254" layer="1"/>
+<wire x1="8.65" y1="25.3" x2="8.85" y2="25.1" width="0.254" layer="1"/>
+<wire x1="8.85" y1="25.1" x2="9.8" y2="25.1" width="0.254" layer="1"/>
+<wire x1="9.8" y1="25.1" x2="10" y2="25.3" width="0.254" layer="1"/>
+<wire x1="6.15" y1="26.3564" x2="6.7936" y2="27" width="0.254" layer="1"/>
+<wire x1="6.7936" y1="27" x2="8.4" y2="27" width="0.254" layer="1"/>
 </signal>
 <signal name="N$2">
 <contactref element="LED" pad="A"/>
 <contactref element="L/EN" pad="1"/>
-<wire x1="5.85" y1="23.95" x2="5.6" y2="24.2" width="0.254" layer="1"/>
-<wire x1="5.6" y1="24.2" x2="5.6" y2="24.9936" width="0.254" layer="1"/>
-<wire x1="5.6" y1="24.9936" x2="5.5936" y2="25" width="0.254" layer="1"/>
-<wire x1="5.85" y1="23.95" x2="7.25" y2="23.95" width="0.254" layer="1"/>
-<wire x1="7.25" y1="23.95" x2="7.55" y2="24.25" width="0.254" layer="1"/>
+<wire x1="6.15" y1="25.5436" x2="7.1936" y2="25.5436" width="0.254" layer="1"/>
+<wire x1="7.1936" y1="25.5436" x2="7.7" y2="26.05" width="0.254" layer="1"/>
 </signal>
 </signals>
