File: board/MINI_SAM_TQFP_2.54_BB_2017_01_17_004.sch (EAGLE design)
At the start: 27 parts, among them J1 MOLEX_47346-100147346, J2 CORTEX_DEBUGPTH, SW1 KMS_SWITCHKMS, SW2 KMS_SWITCHKMS, U1 SAMD21ETQFP, Y1 32.768kHz 7pF

Commit message: Add files via upload
Parts:
- LED: device microbuilder:LED0603_NOOUTLINE -> microbuilder:LED0805_NOOUTLINE
Changed lines of the file:
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@@
 <part name="JP4" library="pinhead+" deviceset="PINHD-1X11" device="1X11_SMT"/>
 <part name="JP3" library="pinhead+" deviceset="PINHD-1X11" device="1X11_SMT"/>
-<part name="LED" library="microbuilder" deviceset="LED" device="0603_NOOUTLINE" value="APT2012LSECK/J3-PRV"/>
+<part name="LED" library="microbuilder" deviceset="LED" device="0805_NOOUTLINE" value="APT2012LSECK/J3-PRV"/>
 <part name="GND14" library="SparkFun-Aesthetics" deviceset="GND" device=""/>
 <part name="IC1" library="Shockley_Custom" deviceset="MCP1700" device=""/>
